Commit message: ajout fichiers launch

File: description/robot.urdf.xacro (robot description, xacro)
@@ -3,3 +3,4 @@
     <xacro:include filename="robot_core.xacro" />
     <xacro:include filename="lidar.xacro" />
+    <xacro:include filename="camera.xacro" />
 </robot>

File: description/robot_core.xacro (robot description, xacro)
@@ -54,9 +54,9 @@
         <visual>
             <geometry>
-                <cylinder radius="0.055" length="0.07"/>
+                <cylinder radius="0.0575" length="0.07"/>
             </geometry>
             <material name="blue"/>
         </visual>
-        <xacro:inertial_cylinder mass="0.1" length="0.07" radius="0.055">
+        <xacro:inertial_cylinder mass="0.1" length="0.07" radius="0.0575">
             <origin xyz="0 0 0" rpy="0 0 0"/>
         </xacro:inertial_cylinder>
@@ -72,9 +72,9 @@
         <visual>
             <geometry>
-                <cylinder radius="0.055" length="0.07"/>
+                <cylinder radius="0.0575" length="0.07"/>
             </geometry>
             <material name="blue"/>
         </visual>
-        <xacro:inertial_cylinder mass="0.1" length="0.07" radius="0.055">
+        <xacro:inertial_cylinder mass="0.1" length="0.07" radius="0.0575">
             <origin xyz="0 0 0" rpy="0 0 0"/>
         </xacro:inertial_cylinder>
@@ -90,9 +90,9 @@
         <visual>
             <geometry>
-                <cylinder radius="0.055" length="0.07"/>
+                <cylinder radius="0.0575" length="0.07"/>
             </geometry>
             <material name="blue"/>
         </visual>
-        <xacro:inertial_cylinder mass="0.1" length="0.07" radius="0.055">
+        <xacro:inertial_cylinder mass="0.1" length="0.07" radius="0.0575">
             <origin xyz="0 0 0" rpy="0 0 0"/>
         </xacro:inertial_cylinder>
@@ -108,9 +108,9 @@
         <visual>
             <geometry>
-                <cylinder radius="0.055" length="0.07"/>
+                <cylinder radius="0.0575" length="0.07"/>
             </geometry>
             <material name="blue"/>
         </visual>
-        <xacro:inertial_cylinder mass="0.1" length="0.07" radius="0.055">
+        <xacro:inertial_cylinder mass="0.1" length="0.07" radius="0.0575">
             <origin xyz="0 0 0" rpy="0 0 0"/>
         </xacro:inertial_cylinder>
