Commit message: changements model

File: description/robot_core.xacro (robot description, xacro)
@@ -13,4 +13,7 @@
     <material name="black">
         <color rgba="0 0 0 1"/>
+    </material>
+    <material name="red">
+        <color rgba="1 0 0 1"/>
     </material>
      <!-- BASE LINK -->
@@ -45,5 +48,5 @@
         <parent link="base_link"/>
         <child link="gh_wheel"/>
-        <origin xyz="0.1 0.1 0" rpy="-${pi/2} 0 0" />
+        <origin xyz="0.1 0.135 0" rpy="-${pi/2} 0 0" />
         <axis xyz="0 0 1"/>
     </joint>
@@ -51,9 +54,9 @@
         <visual>
             <geometry>
-                <cylinder radius="0.055" length="0.04"/>
+                <cylinder radius="0.055" length="0.07"/>
             </geometry>
             <material name="blue"/>
         </visual>
-        <xacro:inertial_cylinder mass="0.1" length="0.04" radius="0.055">
+        <xacro:inertial_cylinder mass="0.1" length="0.07" radius="0.055">
             <origin xyz="0 0 0" rpy="0 0 0"/>
         </xacro:inertial_cylinder>
@@ -63,5 +66,5 @@
         <parent link="base_link"/>
         <child link="gb_wheel"/>
-        <origin xyz="-0.1 0.1 0" rpy="-${pi/2} 0 0" />
+        <origin xyz="-0.1 0.135 0" rpy="-${pi/2} 0 0" />
         <axis xyz="0 0 1"/>
     </joint>
@@ -69,9 +72,9 @@
         <visual>
             <geometry>
-                <cylinder radius="0.055" length="0.04"/>
+                <cylinder radius="0.055" length="0.07"/>
             </geometry>
             <material name="blue"/>
         </visual>
-        <xacro:inertial_cylinder mass="0.1" length="0.04" radius="0.055">
+        <xacro:inertial_cylinder mass="0.1" length="0.07" radius="0.055">
             <origin xyz="0 0 0" rpy="0 0 0"/>
         </xacro:inertial_cylinder>
@@ -81,5 +84,5 @@
         <parent link="base_link"/>
         <child link="dh_wheel"/>
-        <origin xyz="0.1 -0.1 0" rpy="-${pi/2} 0 0" />
+        <origin xyz="0.1 -0.135 0" rpy="-${pi/2} 0 0" />
         <axis xyz="0 0 1"/>
     </joint>
@@ -87,9 +90,9 @@
         <visual>
             <geometry>
-                <cylinder radius="0.055" length="0.04"/>
+                <cylinder radius="0.055" length="0.07"/>
             </geometry>
             <material name="blue"/>
         </visual>
-        <xacro:inertial_cylinder mass="0.1" length="0.04" radius="0.055">
+        <xacro:inertial_cylinder mass="0.1" length="0.07" radius="0.055">
             <origin xyz="0 0 0" rpy="0 0 0"/>
         </xacro:inertial_cylinder>
@@ -99,5 +102,5 @@
         <parent link="base_link"/>
         <child link="db_wheel"/>
-        <origin xyz="-0.1 -0.1 0" rpy="-${pi/2} 0 0" />
+        <origin xyz="-0.1 -0.135 0" rpy="-${pi/2} 0 0" />
         <axis xyz="0 0 1"/>
     </joint>
@@ -105,9 +108,9 @@
         <visual>
             <geometry>
-                <cylinder radius="0.055" length="0.04"/>
+                <cylinder radius="0.055" length="0.07"/>
             </geometry>
             <material name="blue"/>
         </visual>
-        <xacro:inertial_cylinder mass="0.1" length="0.04" radius="0.055">
+        <xacro:inertial_cylinder mass="0.1" length="0.07" radius="0.055">
             <origin xyz="0 0 0" rpy="0 0 0"/>
         </xacro:inertial_cylinder>

Commit message: modif bash

File: description/robot_core.xacro (robot description, xacro)
@@ -45,5 +45,5 @@
     </link>
      <!-- ROUE Gauche Haut GH -->
-     <joint name="gh_wheel_joint" type="continuous">
+     <joint name="gh_wheel_joint" type="fixed">
         <parent link="base_link"/>
         <child link="gh_wheel"/>
@@ -63,5 +63,5 @@
     </link>
      <!-- ROUE GB -->
-     <joint name="gb_wheel_joint" type="continuous">
+     <joint name="gb_wheel_joint" type="fixed">
         <parent link="base_link"/>
         <child link="gb_wheel"/>
@@ -81,5 +81,5 @@
     </link>
     <!-- ROUE DH -->
-    <joint name="dh_wheel_joint" type="continuous">
+    <joint name="dh_wheel_joint" type="fixed">
         <parent link="base_link"/>
         <child link="dh_wheel"/>
@@ -99,5 +99,5 @@
     </link>
     <!-- ROUE DB -->
-    <joint name="db_wheel_joint" type="continuous">
+    <joint name="db_wheel_joint" type="fixed">
         <parent link="base_link"/>
         <child link="db_wheel"/>
